File: Adafruit ESP8266 Feather.sch (EAGLE design)
At the start: 35 parts, among them IC1 CP2104, Q1 mmbt2222, Q2 mmbt2222, SW2 KMR2, U2 SPX3819, U3 MCP73831T-2ACI/OT, X1 JSTPH, X2 ESP-12, X4 20329

Commit message: Finished Schematic: CP2104 + SPX3819 + MCP73831T-2ACI/OT + KMR2(Reset)
Parts:
- removed R6: 4.7K, microbuilder:RESISTOR_0603_NOOUT
Connections:
- new net DTR: IC1G$1.DTR
- new net EN: R7.1, U2.EN
- new net GPIO0: R10.1
- new net N$1: CHG.C, R2.1
- new net N$2: IC1G$1.D+, X4.D+
- new net N$3: R2.2, U3.STAT
- new net N$4: R8.1, U3.PROG
- new net N$6: IC1G$1.D-, X4.D-
- new net N$7: SJ1.1, U3.VBAT
- new net RTS: IC1G$1.RTS
- new net TXD: IC1G$1.RXD
- new net USB_RX: IC1G$1.TXD
- new net VBAT: C3.1, D4.A, SJ1.2, X1.2
- new net VBUS: C6.1, CHG.A, D4.C, IC1G$1.VBUS, R7.2, U2.IN, U3.VDD, X4.VBUS
- net 3.3V: now also C2.1, C7.1, C8.1, D3.A, IC1G$1.REGIN, IC1G$1.VDD, IC1G$1.VIO, U2.OUT; no longer X2.VCC
- net GND: now also C2.2, C3.2, C6.2, C7.2, C8.2, IC1G$1.GND, R8.2, SW2.P, SW2.P1, U2.GND, U3.VSS, X1.1, X4.GND
- net RESET: now also R3.1

Commit message: Schematic: ESP8266 + (JP1 + JP3 I/O Headers)
Parts:
- added R6: 4.7K, microbuilder:RESISTOR_0603_NOOUT
Connections:
- new net ADC: JP1.12, X2.ADC
- new net CH_PD: JP1.1, R1.1, X2.CH_PD
- new net GPIO12/MISO: JP1.4, JP3.5, X2.GPIO12
- new net GPIO13/MOSI: JP1.5, JP3.6, X2.GPIO13
- new net GPIO14/SCK: JP1.6, JP3.4, X2.GPIO14
- new net GPIO15: JP3.7, R6.2, X2.GPIO15
- new net GPIO16: JP3.9, X2.GPIO16
- new net GPIO2: JP3.10, R9.1, X2.GPIO2
- new net GPIO4/SDA: JP3.12, X2.GPIO4
- new net GPIO5/SCL: JP3.11, X2.GPIO5
- new net N$12: Q1.B, R4.2
- new net N$13: Q2.B, R5.2
- new net RXD: JP1.3, R11.2, X2.RXD
- net 3.3V: now also JP1.15, R1.2, R9.2, X2.VCC
- net DTR: now also Q2.E, R4.1
- net EN: now also JP3.2
- net GND: now also JP1.13, R6.1, X2.GND
- net GPIO0: now also JP3.8, Q2.C, X2.GPIO0
- net RESET: now also JP1.16, Q1.C, X2.RESET
- net RTS: now also Q1.E, R5.1
- net TXD: now also JP1.2, X2.TXD
- net USB_RX: now also R11.1
- net VBAT: now also JP3.1
- net VBUS: now also JP3.3

Commit message: Feather .Brd: completed the layout design
Connections:
- net 3.3V: no longer IC1G$1.REGIN, IC1G$1.VDD, IC1G$1.VIO
- net DTR: no longer IC1G$1.DTR
- net GND: no longer IC1G$1.GND
- net N$2: no longer IC1G$1.D+
- net N$6: no longer IC1G$1.D-
- net RTS: no longer IC1G$1.RTS
- net TXD: no longer IC1G$1.RXD
- net USB_RX: no longer IC1G$1.TXD
- net VBUS: no longer IC1G$1.VBUS
